File: hardware/pictas-pcb/pictas.sch (KiCad schematic (older format))
At the start: 26 parts, among them J1 NES_CNT1/2, J10 VizBoard2, J11 VizBoard3, J12 GB, J16 LED_Power_Jack, J2 N64_CNT1/2, J3 N64_CNT3/4, J4 DB1/2, J5 ICSP_VIZ, J6 ICSP_PLAY, J7 USB Port, J8 VizBoard0, J9 VizBoard1, U1 PIC18LF47K42, U2 W25Q128JVS, U3 PIC18F27K42, U5 MCP2221A

Commit message: Revised PCB design again.
Parts:
- added C4, C5: 0.1uF, Capacitor_THT:C_Disc_D3.4mm_W2.1mm_P2.50mm, symbol Device:C_Small
- added J13: RCA Input, pictas:PJRAN1X1U04X, symbol pictas:PJRAN1X1U04X
- added J14: SYNC, Connector_PinHeader_2.54mm:PinHeader_1x03_P2.54mm_Horizontal, symbol Connector_Generic:Conn_01x03
- added J15: CON_RESET, Connector_PinHeader_2.54mm:PinHeader_1x02_P2.54mm_Horizontal, symbol Connector_Generic:Conn_01x02
- added Q1: KSC1815_CON_RESET, digikey-footprints:TO-92-3_Formed_Leads, symbol dk_Transistors-Bipolar-BJT-Single:KSC1815YTA
- added R7: 680k, Resistor_THT:R_Axial_DIN0204_L3.6mm_D1.6mm_P5.08mm_Horizontal, symbol Device:R_Small
- added SW1: MCU_RESET, Button_Switch_THT:SW_PUSH_6mm_H7.3mm, symbol Switch:SW_Push
- added U6: LM1881, Package_SO:SOIC-8_3.9x4.9mm_P1.27mm, symbol pictas:LM1881
- J10: value VizBoard2 -> VIZ_BOARD_3
- J11: value VizBoard3 -> VIZ_BOARD_4
- J16: value LED_Power_Jack -> LED POWER
- J4: value DB1/2 -> DSUB1/2
- J5, J6: footprint Connector_PinHeader_2.54mm:PinHeader_1x05_P2.54mm_Vertical -> Connector_PinHeader_2.54mm:PinHeader_1x05_P2.54mm_Horizontal
- J8: value VizBoard0 -> VIZ_BOARD_1
- J9: value VizBoard1 -> VIZ_BOARD_2
Connections:
- net STROBE0 is gone; now on net STROBE1: J8.2 (Pin_2), U3.4 (RA2)
- net GND: now also J5.1 (Pin_1), J6.1 (Pin_1), C5.1, J13.2, J13.3, J15.1 (Pin_1), R7.2, SW1.1, U6.4 (GND); no longer J5.5 (Pin_5), J6.5 (Pin_5)
- net STROBE1: no longer J9.2 (Pin_2), U3.5 (RA3)
- net STROBE2: now also J9.2 (Pin_2), U3.5 (RA3); no longer J10.2 (Pin_2), U3.6 (RA4)
- net STROBE3: now also J10.2 (Pin_2), U3.6 (RA4); no longer J11.2 (Pin_2), U3.7 (RA5)
- net VDD: now also J5.2 (Pin_2), J6.2 (Pin_2), Q1.1 (E), U6.8 (VCC); no longer J5.4 (Pin_4), J6.4 (Pin_4)
- net MCU_RESET: now reaches R5.1, U1.1 (Vpp/~MCLR~/RE3)
- net MCU_RESET: now also J5.5 (Pin_5), J6.5 (Pin_5), R6.2, U3.1 (Vpp/~MCLR~/RE3), SW1.2; no longer J6.1 (Pin_1)
- net ALT_CLK: now reaches U1.13 (RA7)
- net ALT_CLK: now also J14.2 (Pin_2), U6.3 (VSOUT)
- net CON_RESET: now reaches U1.20 (RD1)
- net CON_RESET: now also Q1.3 (B)
- net OEOUT: now reaches U1.21 (RD2)
- net OEOUT: now also J14.1 (Pin_1), U6.7 (OEOUT)
- net at U1.40 (RB7/ICSPDAT): now also J6.4 (Pin_4); no longer J6.2 (Pin_2)
- net at U3.28 (RB7/ICSPDAT): now also J5.4 (Pin_4); no longer J5.2 (Pin_2)
- net DB11 renamed DSUB11
- net DB12 renamed DSUB12
- net DB13 renamed DSUB13
- net DB14 renamed DSUB14
- net DB15 renamed DSUB15
- net DB16 renamed DSUB16
- net DB17 renamed DSUB17
- net DB21 renamed DSUB21
- net DB22 renamed DSUB22
- net DB23 renamed DSUB23
- net DB24 renamed DSUB24
- net DB25 renamed DSUB25
- net DB26 renamed DSUB26
- net DB27 renamed DSUB27
- new net: C4.1, U6.2 (CVIN)
- new net: C5.2, R7.1, U6.6 (RSET)
- new net: J15.2 (Pin_2), Q1.2 (C)
- new net CVIN: C4.2, J13.1, J14.3 (Pin_3)
- new net STROBE4: J11.2 (Pin_2), U3.7 (RA5)
- no-connect marks 24 -> 27

Commit message: Partially working. SPI to FLASH has severe issues on PCB
Parts:
- removed J13: RCA Input, pictas:PJRAN1X1U04X, symbol pictas:PJRAN1X1U04X
- removed J7: USB Port, Connector_USB:USB_B_OST_USB-B1HSxx_Horizontal, symbol Connector_Generic:Conn_01x04
- removed R5: 10k, Resistor_THT:R_Axial_DIN0204_L3.6mm_D1.6mm_P5.08mm_Horizontal, symbol Device:R
- added J15: USB Port, Connector_USB:USB_B_OST_USB-B1HSxx_Horizontal, symbol Connector:USB_B
- added J16: VIDEO IN, pictas:PJRAN1X1U04X, symbol Connector:Conn_Coaxial
- added J19: AUX_FLASH, Connector_PinHeader_2.54mm:PinHeader_1x04_P2.54mm_Vertical, symbol Connector_Generic:Conn_01x04
- added J7: AUX_VDD_GND_1, Connector_PinHeader_2.54mm:PinHeader_1x02_P2.54mm_Vertical, symbol Connector_Generic:Conn_01x02
- added J8: AUX_VDD_GND_2, Connector_PinSocket_2.54mm:PinSocket_1x02_P2.54mm_Vertical, symbol Connector_Generic:Conn_01x02
- J12: renamed from J3; value N64_CNT3/4 -> N64 3/4
- J2: renamed from J1; value NES_CNT1/2 -> NES 1/2
- J9: renamed from J2; value N64_CNT1/2 -> N64 1/2
- R1, R2: footprint Resistor_THT:R_Axial_DIN0204_L3.6mm_D1.6mm_P5.08mm_Horizontal -> Resistor_THT:R_Axial_DIN0207_L6.3mm_D2.5mm_P10.16mm_Horizontal
- R3: renamed from R6; footprint Resistor_THT:R_Axial_DIN0204_L3.6mm_D1.6mm_P5.08mm_Horizontal -> Resistor_THT:R_Axial_DIN0207_L6.3mm_D2.5mm_P10.16mm_Horizontal
- R4: renamed from R3; footprint Resistor_THT:R_Axial_DIN0204_L3.6mm_D1.6mm_P5.08mm_Horizontal -> Resistor_THT:R_Axial_DIN0207_L6.3mm_D2.5mm_P10.16mm_Horizontal
- R5: renamed from R4; footprint Resistor_THT:R_Axial_DIN0204_L3.6mm_D1.6mm_P5.08mm_Horizontal -> Resistor_THT:R_Axial_DIN0207_L6.3mm_D2.5mm_P10.16mm_Horizontal
- R6: renamed from R7; footprint Resistor_THT:R_Axial_DIN0204_L3.6mm_D1.6mm_P5.08mm_Horizontal -> Resistor_THT:R_Axial_DIN0207_L6.3mm_D2.5mm_P10.16mm_Horizontal
- U4: renamed from U2; value W25Q128JVS -> W25Q128JVSIQ
- renumbered C4 to C3, C3 to C4, J16 to J1, J5 to J10, J15 to J11, J4 to J13, J12 to J14, J6 to J17, J14 to J18, J8 to J3, J9 to J4, J10 to J5, J11 to J6, U3 to U1, U5 to U2, U1 to U3, U6 to U5
Connections:
- net CVIN: now also J16.1 (In)
- net D+: now also U2.13 (D+), J15.3 (D+); no longer U2.12 (D-)
- net D-: now also U2.12 (D-), J15.2 (D-); no longer U2.13 (D+)
- net GND: now also U1.8 (VSS), J15.4 (GND), J15.5 (Shield), J16.2 (Ext), J7.1 (Pin_1), J8.1 (Pin_1)
- net SPI1CS: now also J19.4 (Pin_4)
- net SPI1SCK: now also J19.2 (Pin_2)
- net SPI1SDI: now also J19.1 (Pin_1)
- net SPI1SDO: now also J19.3 (Pin_3)
- net USB_5V: now also J15.1 (VBUS)
- net VDD: now also J7.2 (Pin_2), J8.2 (Pin_2)
- net UART_V2P: now reaches U3.37 (RB4)
- net UART_V2P: now also U1.25 (RB4)
- net UART_P2V: now reaches U3.38 (RB5)
- net UART_P2V: now also U1.26 (RB5)
- net UART-->: no longer names the net of U3.9 (RE1)
- net UART-->: no longer U1.25 (RB4)
- net UART<--: no longer names the net of U3.8 (RE0)
- net UART<--: no longer U1.26 (RB5)
- no-connect marks 27 -> 26
Other:
- moved on the sheet: R3

Commit message: More redesign progress
Parts:
- added C6: 0.1uF, Capacitor_THT:C_Disc_D3.4mm_W2.1mm_P2.50mm, symbol Device:C_Small
- added JP1: VDD_BYPASS, Jumper:SolderJumper-2_P1.3mm_Open_RoundedPad1.0x1.5mm, symbol Jumper:Jumper_2_Open
Connections:
- net GND: now also C6.1
- net SPI1CS: now also J19.3 (Pin_3), U3.34 (RB1); no longer J19.4 (Pin_4), U3.33 (RB0)
- net SPI1SDO: now also J19.4 (Pin_4), U3.33 (RB0); no longer J19.3 (Pin_3), U3.34 (RB1)
- net USB_5V: now also JP1.2 (B)
- net VDD: now also U4.3 (IO2), U4.7 (IO3), C6.2, JP1.1 (A)
- no-connect marks 26 -> 24
Changed lines of the file:
@@
 USB_5V
-Wire Wire Line
-	13250 8125 13350 8125
-NoConn ~ 12250 8325
-NoConn ~ 13250 8225
 Wire Wire Line
 	13550 5375 13650 5375
@@
 Wire Wire Line
 	10150 9400 10250 9400
-Wire Wire Line
-	10900 9500 10150 9500
 $Sheet
 S 9075 9250 1075 400
@@
 	13550 5925 13650 5925
 Wire Wire Line
+	13550 6125 13650 6125
+Wire Wire Line
 	13550 6025 13650 6025
-Wire Wire Line
-	13550 6125 13650 6125
 Text GLabel 13650 5925 2    50   Output ~ 0
 SPI1SCK
+Text GLabel 13650 6125 2    50   Output ~ 0
+SPI1SDO
 Text GLabel 13650 6025 2    50   Output ~ 0
-SPI1SDO
-Text GLabel 13650 6125 2    50   Output ~ 0
 SPI1CS
 Text GLabel 13350 8425 2    50   Output ~ 0
@@
 Wire Wire Line
 	11850 6525 11950 6525
-$Comp
-L power:VDD #PWR033
-U 1 1 617E20B7
-P 13350 8125
-F 0 "#PWR033" H 13350 7975 50  0001 C CNN
-F 1 "VDD" V 13350 8250 50  0000 L CNN
-F 2 "" H 13350 8125 50  0001 C CNN
-F 3 "" H 13350 8125 50  0001 C CNN
-	1    13350 8125
-	0    1    1    0
-$EndComp
-Wire Wire Line
-	12250 8425 12150 8425
-$Comp
-L power:GND #PWR029
-U 1 1 6180D0DC
-P 12150 8425
-F 0 "#PWR029" H 12150 8175 50  0001 C CNN
-F 1 "GND" V 12155 8297 50  0000 R CNN
-F 2 "" H 12150 8425 50  0001 C CNN
-F 3 "" H 12150 8425 50  0001 C CNN
-	1    12150 8425
-	0    1    1    0
-$EndComp
 $Comp
 L power:VDD #PWR032
@@
 Text GLabel 14600 8225 2    50   Output ~ 0
 SPI1SCK
+Text GLabel 14600 8425 2    50   Output ~ 0
+SPI1SDO
 Text GLabel 14600 8325 2    50   Output ~ 0
-SPI1SDO
-Text GLabel 14600 8425 2    50   Output ~ 0
 SPI1CS
 Wire Wire Line
@@
 	14500 8225 14600 8225
 Wire Wire Line
+	14500 8425 14600 8425
+Wire Wire Line
 	14500 8325 14600 8325
-Wire Wire Line
-	14500 8425 14600 8425
 Wire Wire Line
 	5850 6400 6000 6400
@@
 	0    1    1    0
 $EndComp
-Wire Bus Line
-	3550 1400 3550 2100
-Wire Bus Line
-	5500 1400 5500 2100
-Wire Bus Line
-	5800 1400 5800 2100
-Wire Bus Line
-	7750 1400 7750 2100
-Wire Bus Line
-	3875 6800 3875 9275
-Wire Bus Line
-	3250 1025 3250 2100
-Wire Bus Line
-	1400 1025 1400 2100
-Wire Bus Line
-	10075 700  10075 2100
-Wire Bus Line
-	9550 800  9550 2100
-Wire Bus Line
-	8050 800  8050 2100
-Wire Bus Line
-	14825 4025 14825 7575
-Wire Bus Line
-	3250 6800 3250 9950
-Wire Bus Line
-	10675 4025 10675 9400
 Text GLabel 13650 5625 2    50   Output ~ 0
 UART_P2V
@@
 Text Label 11275 10025 2    50   ~ 0
 D-
+Wire Wire Line
+	10900 9500 10150 9500
+Wire Wire Line
+	11400 9500 11500 9500
+$Comp
+L power:VDD #PWR039
+U 1 1 612D2A73
+P 11500 9500
+F 0 "#PWR039" H 11500 9350 50  0001 C CNN
+F 1 "VDD" V 11500 9625 50  0000 L CNN
+F 2 "" H 11500 9500 50  0001 C CNN
+F 3 "" H 11500 9500 50  0001 C CNN
+	1    11500 9500
+	0    1    1    0
+$EndComp
+Wire Wire Line
+	10900 9500 11000 9500
+Connection ~ 10900 9500
+$Comp
+L Jumper:Jumper_2_Open JP1
+U 1 1 612A83CC
+P 11200 9500
+F 0 "JP1" H 11200 9350 50  0000 C CNN
+F 1 "VDD_BYPASS" H 11200 9425 50  0000 C CNN
+F 2 "Jumper:SolderJumper-2_P1.3mm_Open_RoundedPad1.0x1.5mm" H 11200 9500 50  0001 C CNN
+F 3 "~" H 11200 9500 50  0001 C CNN
+	1    11200 9500
+	-1   0    0    1
+$EndComp
+Wire Wire Line
+	12250 8325 12150 8325
+$Comp
+L power:VDD #PWR0102
+U 1 1 61209A62
+P 12150 8325
+F 0 "#PWR0102" H 12150 8175 50  0001 C CNN
+F 1 "VDD" V 12150 8450 50  0000 L CNN
+F 2 "" H 12150 8325 50  0001 C CNN
+F 3 "" H 12150 8325 50  0001 C CNN
+	1    12150 8325
+	0    -1   -1   0
+$EndComp
+$Comp
+L power:GND #PWR029
+U 1 1 6180D0DC
+P 12150 8425
+F 0 "#PWR029" H 12150 8175 50  0001 C CNN
+F 1 "GND" V 12155 8297 50  0000 R CNN
+F 2 "" H 12150 8425 50  0001 C CNN
+F 3 "" H 12150 8425 50  0001 C CNN
+	1    12150 8425
+	0    1    1    0
+$EndComp
+$Comp
+L power:VDD #PWR?
+U 1 1 61481CA6
+P 13350 8225
+F 0 "#PWR?" H 13350 8075 50  0001 C CNN
+F 1 "VDD" V 13350 8350 50  0000 L CNN
+F 2 "" H 13350 8225 50  0001 C CNN
+F 3 "" H 13350 8225 50  0001 C CNN
+	1    13350 8225
+	0    1    1    0
+$EndComp
+Wire Wire Line
+	13250 8225 13350 8225
+Wire Wire Line
+	12150 8425 12250 8425
+Wire Wire Line
+	13250 8125 13300 8125
+$Comp
+L power:VDD #PWR033
+U 1 1 617E20B7
+P 13350 8125
+F 0 "#PWR033" H 13350 7975 50  0001 C CNN
+F 1 "VDD" V 13350 8250 50  0000 L CNN
+F 2 "" H 13350 8125 50  0001 C CNN
+F 3 "" H 13350 8125 50  0001 C CNN
+	1    13350 8125
+	0    1    1    0
+$EndComp
+$Comp
+L Device:C_Small C6
+U 1 1 6132A397
+P 13300 8025
+F 0 "C6" V 13250 8075 38  0000 L CNN
+F 1 "0.1uF" V 13350 8075 38  0000 L CNN
+F 2 "Capacitor_THT:C_Disc_D3.4mm_W2.1mm_P2.50mm" H 13300 8025 50  0001 C CNN
+F 3 "~" H 13300 8025 50  0001 C CNN
+	1    13300 8025
+	-1   0    0    -1
+$EndComp
+Connection ~ 13300 8125
+Wire Wire Line
+	13300 8125 13350 8125
+$Comp
+L power:GND #PWR?
+U 1 1 615F22D9
+P 13350 7875
+F 0 "#PWR?" H 13350 7625 50  0001 C CNN
+F 1 "GND" V 13355 7747 50  0000 R CNN
+F 2 "" H 13350 7875 50  0001 C CNN
+F 3 "" H 13350 7875 50  0001 C CNN
+	1    13350 7875
+	0    -1   -1   0
+$EndComp
+Wire Wire Line
+	13300 7925 13300 7875
+Wire Wire Line
+	13300 7875 13350 7875
+Wire Bus Line
+	3550 1400 3550 2100
+Wire Bus Line
+	5500 1400 5500 2100
+Wire Bus Line
+	5800 1400 5800 2100
+Wire Bus Line
+	7750 1400 7750 2100
+Wire Bus Line
+	3875 6800 3875 9275
+Wire Bus Line
+	3250 1025 3250 2100
+Wire Bus Line
+	1400 1025 1400 2100
+Wire Bus Line
+	10075 700  10075 2100
+Wire Bus Line
+	9550 800  9550 2100
+Wire Bus Line
+	8050 800  8050 2100
+Wire Bus Line
+	14825 4025 14825 7575
+Wire Bus Line
+	3250 6800 3250 9950
+Wire Bus Line
+	10675 4025 10675 9400
 $EndSCHEMATC

Commit message: More design changes
Connections:
- net SPI1SDI: now also J19.4 (Pin_4), U3.33 (RB0), U4.2 (DO(IO1)); no longer J19.1 (Pin_1), U3.36 (RB3), U4.5 (DI(IO0))
- net SPI1SDO: now also J19.1 (Pin_1), U3.36 (RB3), U4.5 (DI(IO0)); no longer J19.4 (Pin_4), U3.33 (RB0), U4.2 (DO(IO1))
Changed lines of the file:
@@
 Wire Wire Line
 	6500 8425 8325 8425
-Text GLabel 13650 5825 2    50   Input ~ 0
-SPI1SDI
 Wire Wire Line
 	13650 5825 13550 5825
@@
 Text GLabel 13650 5925 2    50   Output ~ 0
 SPI1SCK
-Text GLabel 13650 6125 2    50   Output ~ 0
-SPI1SDO
 Text GLabel 13650 6025 2    50   Output ~ 0
 SPI1CS
-Text GLabel 13350 8425 2    50   Output ~ 0
+Text GLabel 12150 8225 0    50   Output ~ 0
 SPI1SDI
 Wire Wire Line
@@
 Text GLabel 12150 8125 0    50   Input ~ 0
 SPI1CS
-Text GLabel 12150 8225 0    50   Input ~ 0
+Text GLabel 13350 8425 2    50   Input ~ 0
 SPI1SDO
 Wire Wire Line
@@
 	-1   0    0    -1
 $EndComp
-Text GLabel 14600 8125 2    50   Input ~ 0
+Text GLabel 14600 8425 2    50   Input ~ 0
 SPI1SDI
 Text GLabel 14600 8225 2    50   Output ~ 0
 SPI1SCK
-Text GLabel 14600 8425 2    50   Output ~ 0
+Text GLabel 14600 8125 2    50   Output ~ 0
 SPI1SDO
 Text GLabel 14600 8325 2    50   Output ~ 0
@@
 $EndComp
 $Comp
-L power:VDD #PWR?
+L power:VDD #PWR0103
 U 1 1 61481CA6
 P 13350 8225
-F 0 "#PWR?" H 13350 8075 50  0001 C CNN
+F 0 "#PWR0103" H 13350 8075 50  0001 C CNN
 F 1 "VDD" V 13350 8350 50  0000 L CNN
 F 2 "" H 13350 8225 50  0001 C CNN
@@
 	13300 8125 13350 8125
 $Comp
-L power:GND #PWR?
+L power:GND #PWR0104
 U 1 1 615F22D9
 P 13350 7875
-F 0 "#PWR?" H 13350 7625 50  0001 C CNN
+F 0 "#PWR0104" H 13350 7625 50  0001 C CNN
 F 1 "GND" V 13355 7747 50  0000 R CNN
 F 2 "" H 13350 7875 50  0001 C CNN
@@
 Wire Bus Line
 	10675 4025 10675 9400
+Text GLabel 13650 6125 2    50   Input ~ 0
+SPI1SDI
+Text GLabel 13650 5825 2    50   Output ~ 0
+SPI1SDO
 $EndSCHEMATC
