File: hardware/pictas-pcb/pictas.kicad_sch (KiCad schematic)
At the start: 40 parts, among them J1 LED POWER, J10 ICSP_VIZ, J11 CON_RESET, J12 N64 3/4, J13 DSUB1/2, J14 GB, J15 USB Port, J16 VIDEO IN, J17 ICSP_PLAY, J18 SYNC, J19 AUX_FLASH, J2 NES 1/2, J3 VIZ_BOARD_1, J4 VIZ_BOARD_2, J5 VIZ_BOARD_3, J6 VIZ_BOARD_4, J7 AUX_VDD_GND_1, J8 AUX_VDD_GND_2, J9 N64 1/2, Q1 KSC1815_CON_RESET, SW1 MCU_RESET, U1 PIC18F27K42, U2 MCP2221A, U3 PIC18LF47K42, U4 W25Q128JVSIQ, U5 LM1881

Commit message: Progress toward replacing pinheaders with D-Sub connector.
Parts:
- removed J10: ICSP_VIZ, Connector_PinHeader_2.54mm:PinHeader_1x05_P2.54mm_Horizontal, symbol Connector_Generic:Conn_01x05
- removed J11: CON_RESET, Connector_PinHeader_2.54mm:PinHeader_1x02_P2.54mm_Horizontal, symbol Connector_Generic:Conn_01x02
- removed J12: N64 3/4, Connector_PinHeader_2.54mm:PinHeader_2x03_P2.54mm_Horizontal, symbol Connector_Generic:Conn_02x03_Odd_Even
- removed J13: DSUB1/2, Connector_PinHeader_2.54mm:PinHeader_2x09_P2.54mm_Horizontal, symbol Connector_Generic:Conn_02x09_Odd_Even
- removed J14: GB, Connector_PinHeader_2.54mm:PinHeader_1x10_P2.54mm_Vertical, symbol Connector_Generic:Conn_01x10
- removed J17: ICSP_PLAY, Connector_PinHeader_2.54mm:PinHeader_1x05_P2.54mm_Horizontal, symbol Connector_Generic:Conn_01x05
- removed J2: NES 1/2, Connector_PinHeader_2.54mm:PinHeader_2x07_P2.54mm_Horizontal, symbol Connector_Generic:Conn_02x07_Odd_Even
- removed J9: N64 1/2, Connector_PinHeader_2.54mm:PinHeader_2x03_P2.54mm_Horizontal, symbol Connector_Generic:Conn_02x03_Odd_Even
- removed JP1: VDD_BYPASS, Jumper:SolderJumper-2_P1.3mm_Open_RoundedPad1.0x1.5mm, symbol Jumper:Jumper_2_Open
- removed Q1: KSC1815_CON_RESET, digikey-footprints:TO-92-3_Formed_Leads, symbol dk_Transistors-Bipolar-BJT-Single:KSC1815YTA
- removed R1, R2, R4, R5: 10k, Resistor_THT:R_Axial_DIN0207_L6.3mm_D2.5mm_P10.16mm_Horizontal, symbol Device:R_Small
- added J12: CONTROLLER_PORT, pictas:L77HDA26SD1CH4R, symbol pictas:DB26_Female_HighDensity_MountingHoles
- added J13: ICSP_PLAY, Connector_PinSocket_2.54mm:PinSocket_1x05_P2.54mm_Horizontal, symbol Connector_Generic:Conn_01x05
- added J8: CON_RESET, Connector_PinHeader_2.54mm:PinHeader_1x03_P2.54mm_Horizontal, symbol Connector_Generic:Conn_01x03
- added J9: ICSP_VIZ, Connector_PinSocket_2.54mm:PinSocket_1x05_P2.54mm_Horizontal, symbol Connector_Generic:Conn_01x05
- added JP1, JP2: SolderJumper_2_Open, Jumper:SolderJumper-2_P1.3mm_Open_TrianglePad1.0x1.5mm, symbol Jumper:SolderJumper_2_Open
- added Q1: BC546, Package_TO_SOT_THT:TO-92_Inline, symbol Transistor_BJT:BC546
- added Q2: BC556, Package_TO_SOT_THT:TO-92_Inline, symbol Transistor_BJT:BC556
- added R2, R3: 1K, Resistor_THT:R_Axial_DIN0207_L6.3mm_D2.5mm_P10.16mm_Horizontal, symbol Device:R
- renumbered J15 to J10, J16 to J11, J18 to J14, J19 to J15, J7 to J2, J8 to J3, J3 to J4, J4 to J5, J5 to J6, J6 to J7, R3 to R1, R6 to R4
Connections:
- net USB_5V is gone; now on net VDD: J10.1 (VBUS)
- net CON_RESET: now also JP1.1 (A), JP2.1 (A), R2.2, R3.2
- net GB8: now also J12.23
- net GND: now also J12.0, J12.26, J12.9, J13.3 (Pin_3), J8.1 (Pin_1), J9.3 (Pin_3), Q2.1 (C)
- net MCU_RESET: now also J13.1 (Pin_1), J9.1 (Pin_1)
- net N64_DATA1: now also J12.6
- net N64_DATA2: now also J12.5
- net N64_DATA3: now also J12.4
- net N64_DATA4: now also J12.3
- net VDD: now also J12.10, J12.19, J13.2 (Pin_2), J9.2 (Pin_2), Q1.1 (C)
- net at U3.39 (RB6/ICSPCLK): now also J13.5 (Pin_5)
- net at U3.40 (RB7/ICSPDAT): now also J13.4 (Pin_4)
- net at U1.27 (RB6/ICSPCLK): now also J9.5 (Pin_5)
- net at U1.28 (RB7/ICSPDAT): now also J9.4 (Pin_4)
- net DSUB11 renamed GB1/DSA1
- net GB1/DSA1: now also J12.12
- net DSUB12 renamed GB2/DSA2
- net GB2/DSA2: now also J12.20
- net DSUB13 renamed GB3/DSA3
- net GB3/DSA3: now also J12.13
- net DSUB14 renamed GB4/DSA4
- net GB4/DSA4: now also J12.21
- net DSUB15 renamed GB5/DSB5
- net GB5/DSB5: now also J12.14
- net DSUB16 renamed GB6/DSB6
- net GB6/DSB6: now also J12.22
- net DSUB17 renamed GB7/DSB7
- net GB7/DSB7: now also J12.15
- net DSUB21 renamed GB9/DSB1/NES_LATCH
- net GB9/DSB1/NES_LATCH: now also J12.18
- net DSUB22 renamed GB10/DSB2/NES_CLK1
- net GB10/DSB2/NES_CLK1: now also J12.8
- net DSUB23 renamed DSB3/NES_DATA1
- net DSB3/NES_DATA1: now also J12.7
- net DSUB24 renamed DSB4/NES_CLK2
- net DSB4/NES_CLK2: now also J12.17
- net DSUB25 renamed DSB5/NES_DATA2
- net DSB5/NES_DATA2: now also J12.16
- net DSUB26 renamed DSB6
- net DSB6: now also J12.24
- net DSUB27 renamed DSB7
- net DSB7: now also J12.25
- net UART_HOST: no longer names the net of U3.10 (RE2)
- net UART_HOST: no longer U1.24 (RB3)
- new net: JP1.2 (B), Q1.2 (B), R2.1
- new net: JP2.2 (B), Q2.2 (B), R3.1
- new net RESET_HI: J8.2 (Pin_2), Q1.3 (E)
- new net RESET_LO: J8.3 (Pin_3), Q2.3 (E)
- no-connect marks 24 -> 26
Other:
- removed sheet Power Select
- note removed: "Board Switching Power Select"
- moved on the sheet: C1, C2, J1, J10, J2, J3, J4, J5, J6, J7, R1, SW1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
